File: PCB/PDM/lm5050_node.kicad_sch (KiCad schematic)
At the start: 5 parts, among them IC12 LM5050MK-1_NOPB, Q2 IAUA250N04S6N007AUMA1

Commit message: Fuck christmas & low side section
Parts:
- IC13: renamed from IC12; footprint SOT95P280X110-6N -> PDM_Additional:SOT95P280X110-6N
- Q3: renamed from Q2; footprint IAUA250N04S6N007AUMA1 -> PDM_Additional:IAUA250N04S6N007AUMA1
- gave numbers to parts that had none: 1
- renumbered C40 to C41, R60 to R61
Changed lines of the file:
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@@
   (symbol (lib_id "power:GND") (at 77.47 40.64 0) (unit 1)
     (in_bom yes) (on_board yes) (fields_autoplaced)
-    (property "Reference" "#PWR?" (id 0) (at 77.47 46.99 0)
+    (property "Reference" "#PWR0169" (id 0) (at 77.47 46.99 0)
       (effects (font (size 1.27 1.27)) hide)
     )
@@
   (symbol (lib_id "power:GND") (at 69.215 71.755 0) (unit 1)
     (in_bom yes) (on_board yes) (fields_autoplaced)
-    (property "Reference" "#PWR0166" (id 0) (at 69.215 78.105 0)
+    (property "Reference" "#PWR0167" (id 0) (at 69.215 78.105 0)
       (effects (font (size 1.27 1.27)) hide)
     )
@@
   (symbol (lib_id "Device:C_Small") (at 77.47 34.925 0) (unit 1)
     (in_bom yes) (on_board yes) (fields_autoplaced)
-    (property "Reference" "C?" (id 0) (at 80.01 33.6612 0)
+    (property "Reference" "C43" (id 0) (at 80.01 33.6612 0)
       (effects (font (size 1.27 1.27)) (justify left))
     )
@@
   (symbol (lib_id "Device:C_Small") (at 70.485 67.945 0) (unit 1)
     (in_bom yes) (on_board yes) (fields_autoplaced)
-    (property "Reference" "C40" (id 0) (at 73.025 66.6812 0)
+    (property "Reference" "C41" (id 0) (at 73.025 66.6812 0)
       (effects (font (size 1.27 1.27)) (justify left))
     )
@@
   (symbol (lib_id "PDM_additional:IAUA250N04S6N007AUMA1") (at 32.385 27.94 0) (unit 1)
     (in_bom yes) (on_board yes) (fields_autoplaced)
-    (property "Reference" "Q2" (id 0) (at 45.085 20.32 0))
+    (property "Reference" "Q3" (id 0) (at 45.085 20.32 0))
     (property "Value" "IAUA250N04S6N007AUMA1" (id 1) (at 45.085 22.86 0))
-    (property "Footprint" "IAUA250N04S6N007AUMA1" (id 2) (at 53.975 25.4 0)
+    (property "Footprint" "PDM_Additional:IAUA250N04S6N007AUMA1" (id 2) (at 53.975 25.4 0)
       (effects (font (size 1.27 1.27)) (justify left) hide)
     )
@@
   (symbol (lib_id "Device:R_Small") (at 60.325 48.26 180) (unit 1)
     (in_bom yes) (on_board yes)
-    (property "Reference" "R60" (id 0) (at 56.515 46.99 0)
+    (property "Reference" "R61" (id 0) (at 56.515 46.99 0)
       (effects (font (size 1.27 1.27)) (justify right))
     )
@@
   (symbol (lib_id "PDM_additional:LM5050MK-1_NOPB") (at 70.485 62.23 270) (mirror x) (unit 1)
     (in_bom yes) (on_board yes)
-    (property "Reference" "IC12" (id 0) (at 65.405 47.625 90)
+    (property "Reference" "IC13" (id 0) (at 65.405 47.625 90)
       (effects (font (size 1.27 1.27)) (justify left))
     )
@@
       (effects (font (size 1.27 1.27)) (justify left))
     )
-    (property "Footprint" "SOT95P280X110-6N" (id 2) (at 73.025 38.1 0)
+    (property "Footprint" "PDM_Additional:SOT95P280X110-6N" (id 2) (at 73.025 38.1 0)
       (effects (font (size 1.27 1.27)) (justify left) hide)
     )
