File: PCB/Tests/VNF1048FTR_TestBoard/VNF1048FTR.kicad_sch (KiCad schematic)
At the start: 25 parts, among them U1 VNF1048FTR

Commit message: VNF1048FTR TestBoard pcb layout change
Parts:
- RS1: footprint Resistor_SMD:R_0402_1005Metric -> Resistor_SMD:R_2512_6332Metric
Changed lines of the file:
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@@
       (effects (font (size 0.8 0.8)))
     )
-    (property "Footprint" "Resistor_SMD:R_0402_1005Metric" (id 2) (at 132.715 69.85 0)
+    (property "Footprint" "Resistor_SMD:R_2512_6332Metric" (id 2) (at 132.715 69.85 0)
       (effects (font (size 1.27 1.27)) hide)
     )

Commit message: Modified test board + gerbers
Parts:
- RH1: footprint Resistor_SMD:R_0805_2012Metric_Pad1.20x1.40mm_HandSolder -> Resistor_THT:R_Axial_DIN0204_L3.6mm_D1.6mm_P2.54mm_Vertical
Connections:
- net DIAG: now also R1.1, R2.1, TP6.1, U1.6 (DIAG)
- net HWLO: now also R7.1, TP7.1, U1.10 (HWLO)
- net HS_GATE: now reaches R9.2, RH1.2, U1.24 (HS_GATE)
- no-connect marks 1 -> 10
Other:
- moved on the sheet: R7
Changed lines of the file:
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@@
   )
   (no_connect (at 126.365 39.37))
+  (no_connect (at 75.565 77.47))
+  (no_connect (at 75.565 59.69))
+  (no_connect (at 75.565 64.77))
+  (no_connect (at 75.565 72.39))
+  (no_connect (at 75.565 74.93))
+  (no_connect (at 126.365 41.91))
+  (no_connect (at 126.365 80.01))
+  (no_connect (at 126.365 57.15))
+  (no_connect (at 126.365 67.31))
   (wire (pts (xy 62.865 52.07) (xy 62.865 52.705))
     (stroke (width 0) (type default) (color 0 0 0 0))
@@
     (stroke (width 0) (type default) (color 0 0 0 0))
   )
-  (wire (pts (xy 73.025 62.23) (xy 74.295 62.23))
+  (wire (pts (xy 71.12 62.23) (xy 74.295 62.23))
     (stroke (width 0) (type default) (color 0 0 0 0))
   )
@@
     (effects (font (size 0.7 0.7)) (justify left bottom))
   )
+  (label "HS_GATE" (at 127 62.23 0)
+    (effects (font (size 0.8 0.8)) (justify left bottom))
+  )
+  (label "HWLO" (at 71.12 62.23 0)
+    (effects (font (size 0.8 0.8)) (justify left bottom))
+  )
   (label "CSN" (at 72.263 41.91 0)
     (effects (font (size 0.8 0.8)) (justify left bottom))
   )
+  (label "DIAG" (at 67.945 52.07 180)
+    (effects (font (size 0.8 0.8)) (justify right bottom))
+  )
   (label "SDI" (at 72.263 44.45 0)
     (effects (font (size 0.8 0.8)) (justify left bottom))
@@
     (effects (font (size 1.27 1.27)) (justify right))
   )
-  (hierarchical_label "HWLO" (shape input) (at 67.945 62.23 180)
+  (hierarchical_label "HWLO" (shape input) (at 66.04 62.23 180)
     (effects (font (size 1.27 1.27)) (justify right))
   )
@@
     (pin "2")
   )
-  (symbol (lib_id "Device:R_Small") (at 70.485 62.23 270) (unit 1)
-    (in_bom yes) (on_board yes)
-    (property "Reference" "R7" (id 0) (at 70.485 62.23 90)
-      (effects (font (size 0.8 0.8)))
-    )
-    (property "Value" "1.2k" (id 1) (at 73.66 63.5 90)
-      (effects (font (size 0.8 0.8)))
-    )
-    (property "Footprint" "Resistor_SMD:R_0402_1005Metric" (id 2) (at 70.485 62.23 0)
-      (effects (font (size 1.27 1.27)) hide)
-    )
-    (property "Datasheet" "~" (id 3) (at 70.485 62.23 0)
+  (symbol (lib_id "Device:R_Small") (at 68.58 62.23 270) (unit 1)
+    (in_bom yes) (on_board yes)
+    (property "Reference" "R7" (id 0) (at 68.58 62.23 90)
+      (effects (font (size 0.8 0.8)))
+    )
+    (property "Value" "1.2k" (id 1) (at 71.755 63.5 90)
+      (effects (font (size 0.8 0.8)))
+    )
+    (property "Footprint" "Resistor_SMD:R_0402_1005Metric" (id 2) (at 68.58 62.23 0)
+      (effects (font (size 1.27 1.27)) hide)
+    )
+    (property "Datasheet" "~" (id 3) (at 68.58 62.23 0)
       (effects (font (size 1.27 1.27)) hide)
     )
@@
       (effects (font (size 0.8 0.8)))
     )
-    (property "Footprint" "Resistor_SMD:R_0805_2012Metric_Pad1.20x1.40mm_HandSolder" (id 2) (at 138.43 62.23 0)
-      (effects (font (size 1.27 1.27)) hide)
-    )
+    (property "Footprint" "Resistor_THT:R_Axial_DIN0204_L3.6mm_D1.6mm_P2.54mm_Vertical" (id 2) (at 138.43 62.23 0)
+      (effects (font (size 1.27 1.27)) hide)
+    )
