File: PCB/Tests/VNF1048FTR_TestBoard/VNF1048FTR_TestBoard.kicad_sch (KiCad schematic)
At the start: 3 parts, among them J1 Conn_01x10_Female, J2 Conn_01x02_Female, Q1 STL135N8F7AG

Commit message: Modified test board + gerbers
Parts:
- removed J1: Conn_01x10_Female, Connector_PinHeader_2.54mm:PinHeader_1x10_P2.54mm_Vertical, symbol Connector:Conn_01x10_Female
- removed J2: Conn_01x02_Female, Connector_AMASS:AMASS_XT30U-M_1x02_P5.0mm_Vertical, symbol Connector:Conn_01x02_Female
- added J1: Conn_01x06_Female, Connector_PinSocket_2.54mm:PinSocket_1x06_P2.54mm_Vertical, symbol Connector:Conn_01x06_Female
- added J2, J3: Conn_01x01_Female, Connector_Wire:SolderWire-2sqmm_1x01_D2mm_OD3.9mm, symbol Connector:Conn_01x01_Female
- added J4: Conn_01x02_Female, Connector_PinSocket_2.54mm:PinSocket_1x02_P2.54mm_Vertical, symbol Connector:Conn_01x02_Female
Connections:
- net +12V: now also J3.1 (Pin_1)
- net +3.3V: now also J4.2 (Pin_2)
- net GND: now also J4.1 (Pin_1)
- net MOS_OUTPUT12V: now also J2.1 (Pin_1)
- net VNF1048FTR/CSN: now also J1.6 (Pin_6)
- net VNF1048FTR/DIAG: now also J1.1 (Pin_1)
- net VNF1048FTR/HWLO: now also J1.2 (Pin_2)
- net VNF1048FTR/SCK: now also J1.3 (Pin_3)
- net VNF1048FTR/SDI: now also J1.5 (Pin_5)
- net VNF1048FTR/SDO: now also J1.4 (Pin_4)
