File: PCB/Tests/BTS50010_TestBoard/BTS50010_TestBoard.kicad_pcb (KiCad board)
At the start: 2 copper layers, 36.6 x 18.8 mm, 10 parts, among them J1 Conn_01x04_Male, U1 BTS50010-1TAE

Commit message: Modfied test board + gerbers
Parts:
- moved C1 7.13 mm to (57.9, 37.6), turned to -90 degrees
- moved R1 1.27 mm to (60.2, 37.6)
- moved R2 0.62 mm to (62.6, 37.6)
- moved C2 0.49 mm to (41.7, 41.2)
Routing:
- net GND: track 49.4 -> 10.5 mm, vias 1 -> 6
- net AUX_IN: track 12.4 -> 9.73 mm
- net Net-(R1-Pad1): track 8.60 -> 9.23 mm
- added copper zone on B.Cu, net GND
- removed copper zone on F.Cu, net GND
- removed copper zone on B.Cu, net IN_VS
- removed copper zone on B.Cu, net OUT_VS
Other:
- board size 36.6 x 18.8 mm -> 37.1 x 21.6 mm
