File: PCB/PDMS/pdms/bts50010.kicad_sch (KiCad schematic)
At the start: 11 parts, among them IC1 BTS500101TAEATMA1

Commit message: Added MCU section
Parts:
- IC1: footprint PG-TO263-7-3_3 -> PDMS_Additional:PG-TO263-7-3_3
Changed lines of the file:
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@@
     (property "Reference" "IC1" (id 0) (at 107.95 43.18 0))
     (property "Value" "BTS500101TAEATMA1" (id 1) (at 107.95 45.72 0))
-    (property "Footprint" "PG-TO263-7-3_3" (id 2) (at 119.38 43.18 0)
+    (property "Footprint" "PDMS_Additional:PG-TO263-7-3_3" (id 2) (at 119.38 43.18 0)
       (effects (font (size 1.27 1.27)) (justify left) hide)
     )

Commit message: Crucial fully assigned schematics
Parts:
- added F2: 40A, PDMS_Additional:0ACA9400TE, symbol Device:Fuse_Small
- C1: footprint (none) -> Capacitor_SMD:C_0402_1005Metric
- C2, C3, C4: footprint (none) -> Capacitor_SMD:C_0805_2012Metric
- D1: value 7V -> 40V; footprint (none) -> Diode_SMD:D_SMA
- R1, R2, R3, R4: footprint (none) -> Resistor_SMD:R_0402_1005Metric
- R5: footprint (none) -> Resistor_SMD:R_0805_2012Metric
Connections:
- net MOS_OUT: now also F2.2; no longer C4.1, IC1.5 (OUT_1), IC1.6 (OUT_2), IC1.7 (OUT_3)
- new net: C4.1, F2.1, IC1.5 (OUT_1), IC1.6 (OUT_2), IC1.7 (OUT_3)
Other:
- note added: "<--Current sense resistor must be accurate!!!"
Changed lines of the file:
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@@
+    (stroke (width 0) (type default) (color 0 0 0 0))
+  )
+  (wire (pts (xy 154.94 55.88) (xy 156.845 55.88))
     (stroke (width 0) (type default) (color 0 0 0 0))
   )
@@
     (stroke (width 0) (type default) (color 0 0 0 0))
   )
-  (wire (pts (xy 129.54 55.88) (xy 132.08 55.88))
+  (wire (pts (xy 129.54 55.88) (xy 149.86 55.88))
     (stroke (width 0) (type default) (color 0 0 0 0))
   )
@@
     (effects (font (size 1.27 1.27) italic) (justify left bottom))
   )
+  (text "<--Current sense resistor must be accurate!!!" (at 93.345 68.58 0)
+    (effects (font (size 0.6 0.6)) (justify left bottom))
+  )
   (text "Pull up/down optional for mechanical switching" (at 60.325 44.45 0)
     (effects (font (size 0.4 0.4)) (justify left bottom))
@@
     (effects (font (size 0.5 0.5)) (justify left bottom))
   )
-  (hierarchical_label "MOS_OUT" (shape output) (at 132.08 55.88 0)
+  (hierarchical_label "MOS_OUT" (shape output) (at 156.845 55.88 0)
     (effects (font (size 1.27 1.27)) (justify left))
   )
@@
       (effects (font (size 1.27 1.27)) (justify left))
     )
-    (property "Footprint" "" (id 2) (at 70.485 52.705 0)
+    (property "Footprint" "Resistor_SMD:R_0402_1005Metric" (id 2) (at 70.485 52.705 0)
       (effects (font (size 1.27 1.27)) hide)
     )
@@
     (property "Reference" "R3" (id 0) (at 82.55 64.135 90))
     (property "Value" "4.7k" (id 1) (at 82.55 66.675 90))
-    (property "Footprint" "" (id 2) (at 82.55 62.23 0)
+    (property "Footprint" "Resistor_SMD:R_0402_1005Metric" (id 2) (at 82.55 62.23 0)
       (effects (font (size 1.27 1.27)) hide)
     )
@@
       (effects (font (size 1.27 1.27)) (justify right))
     )
-    (property "Value" "7V" (id 1) (at 140.97 48.2599 90)
+    (property "Value" "40V" (id 1) (at 140.97 48.2599 90)
       (effects (font (size 1.27 1.27)) (justify right))
     )
-    (property "Footprint" "" (id 2) (at 138.43 46.99 0)
+    (property "Footprint" "Diode_SMD:D_SMA" (id 2) (at 138.43 46.99 0)
       (effects (font (size 1.27 1.27)) hide)
     )
@@
       (effects (font (size 1.27 1.27)) (justify left))
     )
-    (property "Footprint" "" (id 2) (at 129.54 59.69 0)
+    (property "Footprint" "Capacitor_SMD:C_0805_2012Metric" (id 2) (at 129.54 59.69 0)
       (effects (font (size 1.27 1.27)) hide)
     )
@@
       (effects (font (size 1.27 1.27)) (justify left))
     )
-    (property "Footprint" "" (id 2) (at 62.865 52.705 0)
+    (property "Footprint" "Resistor_SMD:R_0402_1005Metric" (id 2) (at 62.865 52.705 0)
       (effects (font (size 1.27 1.27)) hide)
     )
@@
       (effects (font (size 1.27 1.27)) (justify left))
     )
-    (property "Footprint" "" (id 2) (at 91.44 66.04 0)
+    (property "Footprint" "Resistor_SMD:R_0805_2012Metric" (id 2) (at 91.44 66.04 0)
       (effects (font (size 1.27 1.27)) hide)
     )
     (property "Datasheet" "~" (id 3) (at 91.44 66.04 0)
+      (effects (font (size 1.27 1.27)) hide)
+    )
+    (pin "1")
+    (pin "2")
+  )
+  (symbol (lib_id "Device:Fuse_Small") (at 152.4 55.88 0) (unit 1)
+    (in_bom yes) (on_board yes) (fields_autoplaced)
+    (property "Reference" "F2" (id 0) (at 152.4 50.8 0))
+    (property "Value" "40A" (id 1) (at 152.4 53.34 0))
+    (property "Footprint" "PDMS_Additional:0ACA9400TE" (id 2) (at 152.4 55.88 0)
+      (effects (font (size 1.27 1.27)) hide)
+    )
+    (property "Datasheet" "~" (id 3) (at 152.4 55.88 0)
       (effects (font (size 1.27 1.27)) hide)
     )
@@
       (effects (font (size 1.27 1.27)) (justify right))
     )
-    (property "Footprint" "" (id 2) (at 78.74 53.34 0)
+    (property "Footprint" "Capacitor_SMD:C_0805_2012Metric" (id 2) (at 78.74 53.34 0)
       (effects (font (size 1.27 1.27)) hide)
     )
@@
       (effects (font (size 1.27 1.27)) (justify left))
     )
-    (property "Footprint" "" (id 2) (at 76.2 66.04 0)
+    (property "Footprint" "Capacitor_SMD:C_0402_1005Metric" (id 2) (at 76.2 66.04 0)
       (effects (font (size 1.27 1.27)) hide)
     )
@@
     (property "Reference" "R4" (id 0) (at 88.9 59.69 90))
     (property "Value" "4.7k" (id 1) (at 88.9 54.61 90))
-    (property "Footprint" "" (id 2) (at 88.9 57.15 0)
+    (property "Footprint" "Resistor_SMD:R_0402_1005Metric" (id 2) (at 88.9 57.15 0)
       (effects (font (size 1.27 1.27)) hide)
     )
@@
       (effects (font (size 1.27 1.27)) (justify left))
     )
-    (property "Footprint" "" (id 2) (at 127 48.26 0)
-      (effects (font (size 1.27 1.27)) hide)
-    )
+    (property "Footprint" "Capacitor_SMD:C_0805_2012Metric" (id 2) (at 127 48.26 0)
+      (effects (font (size 1.27 1.27)) hide)
+    )
