File: PCB/PDMS/pdms/bts50010.kicad_sch (KiCad schematic)
At the start: 13 parts, among them IC1 BTS500101TAEATMA1

Commit message: HS section layout
Connections:
- net IN: now reaches IC1.2 (IN), R4.2
- net IS: now reaches IC1.3 (IS), R3.1, R5.1
Changed lines of the file:
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@@
     (effects (font (size 0.5 0.5)) (justify left bottom))
+  )
+  (label "IS" (at 92.71 62.23 0)
+    (effects (font (size 1.27 1.27)) (justify left bottom))
+  )
+  (label "IN" (at 92.71 57.15 0)
+    (effects (font (size 1.27 1.27)) (justify left bottom))
   )
   (label "OUT" (at 135.89 55.88 0)

Commit message: Before disaster
Parts:
- C2: footprint Capacitor_SMD:C_0603_1608Metric -> Capacitor_SMD:C_0402_1005Metric
Connections:
- net IN: now also C2.1, R1.2, R2.2
- net SIG_IN: no longer C2.1, R1.2, R2.2
Other:
- moved on the sheet: C2
Changed lines of the file:
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@@
   (junction (at 124.46 59.69) (diameter 0) (color 0 0 0 0)
   )
+  (junction (at 83.185 57.15) (diameter 0) (color 0 0 0 0)
+  )
   (junction (at 70.485 57.15) (diameter 0) (color 0 0 0 0)
   )
@@
   (junction (at 124.46 55.88) (diameter 0) (color 0 0 0 0)
   )
-  (junction (at 78.74 57.15) (diameter 0) (color 0 0 0 0)
-  )
   (junction (at 138.43 52.07) (diameter 0) (color 0 0 0 0)
   )
@@
     (stroke (width 0) (type default) (color 0 0 0 0))
   )
-  (wire (pts (xy 58.42 57.15) (xy 62.865 57.15))
-    (stroke (width 0) (type default) (color 0 0 0 0))
-  )
-  (wire (pts (xy 91.44 57.15) (xy 93.98 57.15))
+  (wire (pts (xy 48.26 57.15) (xy 51.435 57.15))
+    (stroke (width 0) (type default) (color 0 0 0 0))
+  )
+  (wire (pts (xy 56.515 57.15) (xy 62.865 57.15))
+    (stroke (width 0) (type default) (color 0 0 0 0))
+  )
+  (wire (pts (xy 83.185 57.15) (xy 93.98 57.15))
     (stroke (width 0) (type default) (color 0 0 0 0))
   )
@@
     (stroke (width 0) (type default) (color 0 0 0 0))
   )
-  (wire (pts (xy 86.36 57.15) (xy 78.74 57.15))
-    (stroke (width 0) (type default) (color 0 0 0 0))
-  )
   (wire (pts (xy 127 52.07) (xy 138.43 52.07))
     (stroke (width 0) (type default) (color 0 0 0 0))
@@
     (stroke (width 0) (type default) (color 0 0 0 0))
   )
-  (wire (pts (xy 78.74 57.15) (xy 78.74 55.88))
+  (wire (pts (xy 83.185 57.15) (xy 83.185 55.88))
     (stroke (width 0) (type default) (color 0 0 0 0))
   )
@@
     (stroke (width 0) (type default) (color 0 0 0 0))
   )
-  (wire (pts (xy 70.485 57.15) (xy 78.74 57.15))
+  (wire (pts (xy 70.485 57.15) (xy 83.185 57.15))
     (stroke (width 0) (type default) (color 0 0 0 0))
   )
@@
     (stroke (width 0) (type default) (color 0 0 0 0))
   )
-  (wire (pts (xy 78.74 49.53) (xy 78.74 50.8))
+  (wire (pts (xy 83.185 49.53) (xy 83.185 50.8))
     (stroke (width 0) (type default) (color 0 0 0 0))
   )
@@
     (effects (font (size 1.27 1.27)) (justify left))
   )
-  (hierarchical_label "SIG_IN" (shape input) (at 58.42 57.15 180)
+  (hierarchical_label "SIG_IN" (shape input) (at 48.26 57.15 180)
     (effects (font (size 1.27 1.27)) (justify right))
   )
@@
     (pin "1")
   )
-  (symbol (lib_id "Device:C_Small") (at 78.74 53.34 180) (unit 1)
-    (in_bom yes) (on_board yes)
-    (property "Reference" "C2" (id 0) (at 81.28 51.435 0)
+  (symbol (lib_id "Device:C_Small") (at 83.185 53.34 180) (unit 1)
+    (in_bom yes) (on_board yes)
+    (property "Reference" "C2" (id 0) (at 85.725 51.435 0)
       (effects (font (size 1.27 1.27)) (justify right))
     )
-    (property "Value" "150nF" (id 1) (at 80.645 53.975 0)
+    (property "Value" "150nF" (id 1) (at 85.09 53.975 0)
       (effects (font (size 1.27 1.27)) (justify right))
     )
-    (property "Footprint" "Capacitor_SMD:C_0603_1608Metric" (id 2) (at 78.74 53.34 0)
-      (effects (font (size 1.27 1.27)) hide)
-    )
-    (property "Datasheet" "~" (id 3) (at 78.74 53.34 0)
+    (property "Footprint" "Capacitor_SMD:C_0402_1005Metric" (id 2) (at 83.185 53.34 0)
+      (effects (font (size 1.27 1.27)) hide)
+    )
+    (property "Datasheet" "~" (id 3) (at 83.185 53.34 0)
       (effects (font (size 1.27 1.27)) hide)
     )
@@
     (pin "2")
   )
-  (symbol (lib_id "Device:R_Small") (at 88.9 57.15 90) (unit 1)
-    (in_bom yes) (on_board yes)
-    (property "Reference" "R4" (id 0) (at 88.9 59.69 90))
-    (property "Value" "4.7k" (id 1) (at 88.9 54.61 90))
-    (property "Footprint" "Resistor_SMD:R_0402_1005Metric" (id 2) (at 88.9 57.15 0)
-      (effects (font (size 1.27 1.27)) hide)
-    )
-    (property "Datasheet" "~" (id 3) (at 88.9 57.15 0)
-      (effects (font (size 1.27 1.27)) hide)
-    )
-    (pin "1")
-    (pin "2")
-  )
   (symbol (lib_id "Device:C_Small") (at 127 48.26 0) (unit 1)
     (in_bom yes) (on_board yes)
@@
     (pin "2")
   )
-  (symbol (lib_id "power:GND") (at 78.74 49.53 180) (unit 1)
-    (in_bom yes) (on_board yes)
-    (property "Reference" "#PWR0106" (id 0) (at 78.74 43.18 0)
-      (effects (font (size 1.27 1.27)) hide)
-    )
-    (property "Value" "GND" (id 1) (at 78.74 45.72 0))
-    (property "Footprint" "" (id 2) (at 78.74 49.53 0)
-      (effects (font (size 1.27 1.27)) hide)
-    )
-    (property "Datasheet" "" (id 3) (at 78.74 49.53 0)
-      (effects (font (size 1.27 1.27)) hide)
-    )
-    (pin "1")
+  (symbol (lib_id "power:GND") (at 83.185 49.53 180) (unit 1)
+    (in_bom yes) (on_board yes)
+    (property "Reference" "#PWR0106" (id 0) (at 83.185 43.18 0)
+      (effects (font (size 1.27 1.27)) hide)
+    )
+    (property "Value" "GND" (id 1) (at 83.185 45.72 0))
+    (property "Footprint" "" (id 2) (at 83.185 49.53 0)
+      (effects (font (size 1.27 1.27)) hide)
+    )
+    (property "Datasheet" "" (id 3) (at 83.185 49.53 0)
+      (effects (font (size 1.27 1.27)) hide)
+    )
+    (pin "1")
+  )
+  (symbol (lib_id "Device:R_Small") (at 53.975 57.15 90) (unit 1)
+    (in_bom yes) (on_board yes)
+    (property "Reference" "R4" (id 0) (at 53.975 59.69 90))
+    (property "Value" "4.7k" (id 1) (at 53.975 54.61 90))
+    (property "Footprint" "Resistor_SMD:R_0402_1005Metric" (id 2) (at 53.975 57.15 0)
+      (effects (font (size 1.27 1.27)) hide)
+    )
+    (property "Datasheet" "~" (id 3) (at 53.975 57.15 0)
+      (effects (font (size 1.27 1.27)) hide)
+    )
+    (pin "1")
+    (pin "2")
   )
   (symbol (lib_id "power:+12V") (at 62.865 49.53 0) (unit 1)

Commit message: Safety finished - 53
Connections:
- net +12V: no longer R1.1
- new net +3.3V: R1.1
Changed lines of the file:
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@@
+    (pin "1")
+  )
+  (symbol (lib_id "power:+3.3V") (at 62.865 49.53 0) (unit 1)
+    (in_bom yes) (on_board yes) (fields_autoplaced)
+    (property "Reference" "#PWR?" (id 0) (at 62.865 53.34 0)
+      (effects (font (size 1.27 1.27)) hide)
+    )
+    (property "Value" "+3.3V" (id 1) (at 62.865 44.45 0))
+    (property "Footprint" "" (id 2) (at 62.865 49.53 0)
+      (effects (font (size 1.27 1.27)) hide)
+    )
+    (property "Datasheet" "" (id 3) (at 62.865 49.53 0)
+      (effects (font (size 1.27 1.27)) hide)
+    )
     (pin "1")
   )
@@
     (pin "2")
   )
-  (symbol (lib_id "power:+12V") (at 62.865 49.53 0) (unit 1)
-    (in_bom yes) (on_board yes)
-    (property "Reference" "#PWR0109" (id 0) (at 62.865 53.34 0)
-      (effects (font (size 1.27 1.27)) hide)
-    )
-    (property "Value" "+12V" (id 1) (at 62.865 45.72 0))
-    (property "Footprint" "" (id 2) (at 62.865 49.53 0)
-      (effects (font (size 1.27 1.27)) hide)
-    )
-    (property "Datasheet" "" (id 3) (at 62.865 49.53 0)
-      (effects (font (size 1.27 1.27)) hide)
-    )
-    (pin "1")
-  )
   (symbol (lib_id "power:GND") (at 91.44 50.165 180) (unit 1)

Commit message: Minor changes in annotations
Other:
- note added: "This acts as voltage divider !!!!!! ↓→"
Changed lines of the file:
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@@
     (effects (font (size 0.6 0.6)) (justify left bottom))
+  )
+  (text "This acts as voltage divider !!!!!! ↓→\n                                    "
+    (at 24.13 109.855 0)
+    (effects (font (size 1.27 1.27) (thickness 0.254) bold italic) (justify left bottom))
   )
   (text "Pull up/down optional for mechanical switching" (at 60.325 44.45 0)
@@
   )
   (symbol (lib_id "power:+3.3V") (at 62.865 49.53 0) (unit 1)
-    (in_bom yes) (on_board yes) (fields_autoplaced)
+    (in_bom yes) (on_board yes)
     (property "Reference" "#PWR0109" (id 0) (at 62.865 53.34 0)
       (effects (font (size 1.27 1.27)) hide)
     )
-    (property "Value" "+3.3V" (id 1) (at 62.865 44.45 0))
+    (property "Value" "+3.3V" (id 1) (at 62.865 45.72 0))
     (property "Footprint" "" (id 2) (at 62.865 49.53 0)
       (effects (font (size 1.27 1.27)) hide)
