File: PCB/PDMS/pdms/pdms.kicad_pcb (KiCad board)
At the start: 4 copper layers, 328 parts, among them IC1 BTS500101TAEATMA1, IC10 LDO40LPU50RY, IC11 MP2332HGTL-P, IC12 TMP126NDCKR, IC14 TMP126NDCKR, IC15 LM74700MDDFREP, IC16 BTS722204ESAXUMA1, IC17 ASM330LHHTR, IC18 NX3L4051PW,118, IC19 STM32L496ZGT6, IC2 BTS500101TAEATMA1, IC20 AT25SF128A-SHB-T, IC3 BTS500101TAEATMA1, IC4 BTS500101TAEATMA1, IC5 BTS500101TAEATMA1, IC6 BTS500101TAEATMA1, IC7 BTS722204ESAXUMA1, IC8 BTS500101TAEATMA1, IC9 BTS500101TAEATMA1, J1 DBG, J2 6473427-1, Q1 AO3401A, Q2 MMBT3904, Q3 IAUA250N04S6N007AUMA1, U1 CPC1117N, U10 CPC1117N, U2 MCP2561-E-SN, U3 MCP2561-E-SN, U4 CPC1117N, U5 CPC1117N, U6 CPC1117N, U7 CPC1117N, U8 CPC1117N, U9 CPC1117N, Y1 48Mhz, Y2 32KHz

Commit message: Added voltage mux section & layouting high side - hp
Parts:
- added C89: 100nF, Capacitor_SMD:C_0402_1005Metric_Pad0.74x0.62mm_HandSolder, F.Cu at (446.0, 217.8)
- added IC13: NX3L4051PW,118, PDMS_Additional:SOP65P640X110-16N, F.Cu at (448.9, 213.5)
- added R134: 2.3k, Resistor_SMD:R_0402_1005Metric, F.Cu at (454.8, 215.1)
- added R135: 10, Resistor_SMD:R_0402_1005Metric, F.Cu at (454.8, 213.1)
- added R136: 10k, Resistor_SMD:R_0402_1005Metric, F.Cu at (445.9, 219.8)
- added R137: 10k, Resistor_SMD:R_0402_1005Metric, F.Cu at (445.9, 221.8)
- added R138: 10k, Resistor_SMD:R_0402_1005Metric, F.Cu at (452.0, 217.8)
- added R139: 10k, Resistor_SMD:R_0402_1005Metric, F.Cu at (454.8, 211.1)
- added R140: 10k, Resistor_SMD:R_0402_1005Metric, F.Cu at (445.9, 223.8)
- added R141: 10k, Resistor_SMD:R_0402_1005Metric, F.Cu at (448.8, 219.8)
- added R142: 10k, Resistor_SMD:R_0402_1005Metric, F.Cu at (449.1, 217.8)
- added R143: 10k, Resistor_SMD:R_0402_1005Metric, F.Cu at (457.7, 211.1)
- added R144: 1R, Resistor_SMD:R_0805_2012Metric, F.Cu at (31.1, 74.4)
- added R145: 1R, Resistor_SMD:R_0805_2012Metric, F.Cu at (712.2, 143.1)
- added R146: 1R, Resistor_SMD:R_0805_2012Metric, F.Cu at (673.5, 101.5)
- added R147: 1R, Resistor_SMD:R_0805_2012Metric, F.Cu at (629.1, 184.7)
- added R148: 1R, Resistor_SMD:R_0805_2012Metric, F.Cu at (546.0, 309.5)
- added R149: 1R, Resistor_SMD:R_0805_2012Metric, F.Cu at (546.0, 267.9)
- added R150: 1R, Resistor_SMD:R_0805_2012Metric, F.Cu at (629.1, 226.3)
- added R151: 1R, Resistor_SMD:R_0805_2012Metric, F.Cu at (712.2, 184.7)
- C10, C2, C21, C25, C29, C33, C37, C6: footprint Capacitor_SMD:C_0805_2012Metric -> Capacitor_SMD:C_0603_1608Metric
- R10, R15, R32, R37, R42, R48, R5, R53: footprint Resistor_SMD:R_0805_2012Metric -> Resistor_SMD:R_0402_1005Metric
- moved C33 620.5 mm to (632.7, 221.8), turned to 0 degrees
- moved R43 619.8 mm to (626.8, 228.8), turned to 0 degrees
- moved R46 617.0 mm to (636.4, 221.3), turned to 0 degrees
- moved IC9 615.8 mm to (699.6, 183.9), turned to 0 degrees
- moved R45 610.2 mm to (623.9, 228.8), turned to 0 degrees
- moved R48 610.1 mm to (622.9, 238.9), turned to 0 degrees
- moved R47 609.9 mm to (623.9, 230.8), turned to 0 degrees
- moved D8 608.7 mm to (626.4, 222.5), turned to 0 degrees
- moved C32 608.1 mm to (623.9, 232.8), turned to 0 degrees
- moved C34 606.9 mm to (624.6, 226.3), turned to 0 degrees
- moved F8 597.1 mm to (615.7, 240.6), turned to 0 degrees
- moved C35 594.5 mm to (612.8, 245.2), turned to 0 degrees
- moved C21 593.8 mm to (632.7, 180.2), turned to 0 degrees
- moved R16 592.7 mm to (626.8, 187.2), turned to 0 degrees
- moved IC8 590.7 mm to (616.5, 225.5), turned to 0 degrees
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Connections:
- net Net-(C12-Pad1) renamed /POWER_SWITCHES/BTS50010-1TAE2/OUT
- net Net-(C23-Pad1) renamed /POWER_SWITCHES/BTS50010-1TAE3/OUT
- net Net-(C27-Pad1) renamed /POWER_SWITCHES/BTS50010-1TAE4/OUT
- net Net-(C31-Pad1) renamed /POWER_SWITCHES/BTS50010-1TAE6/OUT
- net Net-(C35-Pad1) renamed /POWER_SWITCHES/BTS50010-1TAE7/OUT
- net Net-(C39-Pad1) renamed /POWER_SWITCHES/BTS50010-1TAE5/OUT
- net Net-(C4-Pad1) renamed /POWER_SWITCHES/BTS50010-1TAE/OUT
- net Net-(C8-Pad1) renamed /POWER_SWITCHES/BTS50010-1TAE1/OUT
- D1 pad 2: GND -> Net-(D1-Pad2)
- D2 pad 2: GND -> Net-(D2-Pad2)
- D3 pad 2: GND -> Net-(D3-Pad2)
- D5 pad 2: GND -> Net-(D5-Pad2)
- D6 pad 2: GND -> Net-(D6-Pad2)
- D7 pad 2: GND -> Net-(D7-Pad2)
- D8 pad 2: GND -> Net-(D8-Pad2)
- D9 pad 2: GND -> Net-(D9-Pad2)
- IC14 pad 5: /PERIPHERAL/TEMP1_ALERT -> /PERIPHERAL/TEMP2_ALERT
- IC19 pad 11: unconnected-(IC19-Pad11) -> /NTC_SECTION/NTC_SEL1
- IC19 pad 118: /TEMP2_ALERT -> /PERIPHERAL/TEMP2_ALERT
- IC19 pad 12: /NTC_SECTION/NTC_SEL1 -> /NTC_SECTION/NTC_SEL2
- IC19 pad 13: /NTC_SECTION/NTC_SEL2 -> /NTC_SECTION/NTC_SEL3
- IC19 pad 14: /NTC_SECTION/NTC_SEL3 -> unconnected-(IC19-Pad14)
- IC19 pad 2: unconnected-(IC19-Pad2) -> /VOLTAGE_OUT_MUX/HP_MOS_SEL1
- IC19 pad 20: unconnected-(IC19-Pad20) -> /VOLTAGE_OUT_MUX/HP_MOS_ADC
- IC19 pad 3: unconnected-(IC19-Pad3) -> /VOLTAGE_OUT_MUX/HP_MOS_SEL2
- IC19 pad 4: unconnected-(IC19-Pad4) -> /VOLTAGE_OUT_MUX/HP_MOS_SEL3
- R67 pad 2: /PERIPHERAL/TEMP1_ALERT -> /PERIPHERAL/TEMP2_ALERT
Routing:
- net GND: track 0.00 -> 3.37 mm, vias 0 -> 1
- net Net-(IC1-Pad2): track 0.00 -> 3.18 mm, vias 0 -> 1
- net Net-(IC1-Pad3): track 0.00 -> 3.15 mm, vias 0 -> 1
- added copper zone on F.Cu, net /POWER_SWITCHES/BTS50010-1TAE/OUT
- added copper zone on In1.Cu, net /POWER_SWITCHES/BTS50010-1TAE/OUT
Other:
- board outline added: 126.1 x 81.2 mm

Commit message: HS section layout
Parts:
- added R152: 2.3k, Resistor_SMD:R_0402_1005Metric, F.Cu at (392.4, 109.9)
- added R153: 2.3k, Resistor_SMD:R_0402_1005Metric, F.Cu at (389.2, 115.8)
- added R154: 10k, Resistor_SMD:R_0402_1005Metric, F.Cu at (392.1, 115.8)
- added R155: 10k, Resistor_SMD:R_0402_1005Metric, F.Cu at (401.0, 103.1)
- added R156: 2.3k, Resistor_SMD:R_0402_1005Metric, F.Cu at (403.9, 103.1)
- added R157: 2.3k, Resistor_SMD:R_0402_1005Metric, F.Cu at (401.0, 105.1)
- added R158: 10k, Resistor_SMD:R_0402_1005Metric, F.Cu at (398.2, 109.1)
- R134: value 2.3k -> 10k
- R137, R138, R140, R141: value 10k -> 2.3k
- moved R8 679.7 mm to (43.1, 70.9)
- moved C6 676.2 mm to (40.9, 96.0)
- moved R6 675.0 mm to (36.7, 95.3), turned to 180 degrees
- moved R7 671.9 mm to (36.7, 99.1), turned to 180 degrees
- moved R145 669.5 mm to (46.2, 74.7), turned to -90 degrees
- moved C5 668.7 mm to (43.1, 69.6), turned to 180 degrees
- moved R9 668.2 mm to (40.5, 99.1), turned to 180 degrees
- moved R10 668.2 mm to (43.1, 72.1)
- moved F3 667.9 mm to (36.7, 69.0), turned to 90 degrees
- moved D2 666.0 mm to (46.2, 80.1), turned to 90 degrees
- moved C7 664.1 mm to (46.2, 85.0), turned to 180 degrees
- moved IC2 663.4 mm to (38.6, 85.7), turned to 180 degrees
- moved C8 662.3 mm to (40.0, 70.5)
- moved R13 623.1 mm to (58.2, 70.9)
- moved C10 621.0 mm to (56.1, 96.0)
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Connections:
- net Net-(IC1-Pad2) renamed /POWER_SWITCHES/BTS50010-1TAE/IN
- net Net-(IC1-Pad3) renamed /POWER_SWITCHES/BTS50010-1TAE/IS
- net Net-(IC2-Pad2) renamed /POWER_SWITCHES/BTS50010-1TAE1/IN
- net Net-(IC2-Pad3) renamed /POWER_SWITCHES/BTS50010-1TAE1/IS
- net Net-(IC3-Pad2) renamed /POWER_SWITCHES/BTS50010-1TAE2/IN
- net Net-(IC3-Pad3) renamed /POWER_SWITCHES/BTS50010-1TAE2/IS
- net Net-(IC4-Pad2) renamed /POWER_SWITCHES/BTS50010-1TAE3/IN
- net Net-(IC4-Pad3) renamed /POWER_SWITCHES/BTS50010-1TAE3/IS
- net Net-(IC5-Pad2) renamed /POWER_SWITCHES/BTS50010-1TAE4/IN
- net Net-(IC5-Pad3) renamed /POWER_SWITCHES/BTS50010-1TAE4/IS
- net Net-(IC6-Pad2) renamed /POWER_SWITCHES/BTS50010-1TAE6/IN
- net Net-(IC6-Pad3) renamed /POWER_SWITCHES/BTS50010-1TAE6/IS
- net Net-(IC8-Pad2) renamed /POWER_SWITCHES/BTS50010-1TAE7/IN
- net Net-(IC8-Pad3) renamed /POWER_SWITCHES/BTS50010-1TAE7/IS
- net Net-(IC9-Pad2) renamed /POWER_SWITCHES/BTS50010-1TAE5/IN
- net Net-(IC9-Pad3) renamed /POWER_SWITCHES/BTS50010-1TAE5/IS
- R134 pad 1: GND -> Net-(IC13-Pad4)
- R134 pad 2: /VOLTAGE_OUT_MUX/HP_MOS_ADC -> HP_MOS8
- R137 pad 1: Net-(IC13-Pad14) -> GND
- R137 pad 2: HP_MOS2 -> Net-(IC13-Pad4)
- R138 pad 1: Net-(IC13-Pad15) -> GND
- R138 pad 2: HP_MOS3 -> Net-(IC13-Pad13)
- R139 pad 1: Net-(IC13-Pad12) -> Net-(IC13-Pad2)
- R139 pad 2: HP_MOS4 -> HP_MOS7
- R140 pad 1: Net-(IC13-Pad1) -> GND
- R140 pad 2: HP_MOS5 -> Net-(IC13-Pad2)
- R141 pad 1: Net-(IC13-Pad5) -> GND
- R141 pad 2: HP_MOS6 -> Net-(IC13-Pad14)
- R142 pad 1: Net-(IC13-Pad2) -> Net-(IC13-Pad14)
- R142 pad 2: HP_MOS7 -> HP_MOS2
- R143 pad 1: Net-(IC13-Pad4) -> Net-(IC13-Pad5)
- R143 pad 2: HP_MOS8 -> HP_MOS6
Routing:
- net GND: track 3.37 -> 241.9 mm, vias 1 -> 290
- net /POWER_SWITCHES/BTS50010-1TAE4/IS: track 0.00 -> 31.5 mm
- net /POWER_SWITCHES/BTS50010-1TAE1/IS: track 0.00 -> 31.5 mm
- net /POWER_SWITCHES/BTS50010-1TAE7/IS: track 0.00 -> 31.5 mm
- net /POWER_SWITCHES/BTS50010-1TAE6/IS: track 0.00 -> 31.5 mm
- net /POWER_SWITCHES/BTS50010-1TAE3/IS: track 0.00 -> 31.5 mm
- net /POWER_SWITCHES/BTS50010-1TAE2/IS: track 0.00 -> 31.5 mm
- net /POWER_SWITCHES/BTS50010-1TAE5/IS: track 0.00 -> 31.5 mm
- net /POWER_SWITCHES/BTS50010-1TAE7/IN: track 0.00 -> 12.7 mm, vias 0 -> 4
- net /POWER_SWITCHES/BTS50010-1TAE6/IN: track 0.00 -> 12.7 mm, vias 0 -> 4
- net /POWER_SWITCHES/BTS50010-1TAE2/IN: track 0.00 -> 12.7 mm, vias 0 -> 4
- net /POWER_SWITCHES/BTS50010-1TAE4/IN: track 0.00 -> 12.7 mm, vias 0 -> 4
- net /POWER_SWITCHES/BTS50010-1TAE1/IN: track 0.00 -> 12.7 mm, vias 0 -> 4
- net /POWER_SWITCHES/BTS50010-1TAE5/IN: track 0.00 -> 12.7 mm, vias 0 -> 4
- net /POWER_SWITCHES/BTS50010-1TAE3/IN: track 0.00 -> 12.7 mm, vias 0 -> 4
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- added copper zone on F.Cu, net +12V
- added copper zone on In1.Cu, net +12V
- added copper zone on F.Cu, net /POWER_SWITCHES/BTS50010-1TAE1/OUT
- added copper zone on In1.Cu, net /POWER_SWITCHES/BTS50010-1TAE1/OUT
- added copper zone on F.Cu, net /POWER_SWITCHES/BTS50010-1TAE2/OUT
- added copper zone on In1.Cu, net /POWER_SWITCHES/BTS50010-1TAE2/OUT
- added copper zone on F.Cu, net /POWER_SWITCHES/BTS50010-1TAE3/OUT
- added copper zone on In1.Cu, net /POWER_SWITCHES/BTS50010-1TAE3/OUT
- added copper zone on F.Cu, net /POWER_SWITCHES/BTS50010-1TAE4/OUT
- added copper zone on In1.Cu, net /POWER_SWITCHES/BTS50010-1TAE4/OUT
- added copper zone on F.Cu, net /POWER_SWITCHES/BTS50010-1TAE5/OUT
- added copper zone on In1.Cu, net /POWER_SWITCHES/BTS50010-1TAE5/OUT
- added copper zone on F.Cu, net /POWER_SWITCHES/BTS50010-1TAE6/OUT
- added copper zone on In1.Cu, net /POWER_SWITCHES/BTS50010-1TAE6/OUT
- added copper zone on F.Cu, net /POWER_SWITCHES/BTS50010-1TAE7/OUT
- added copper zone on In1.Cu, net /POWER_SWITCHES/BTS50010-1TAE7/OUT
- added copper zone on F.Cu, net GND
- added copper zone on In2.Cu, net GND

Commit message: Welcome back
Connections:
- F9 pad 2: HP_MOS7 -> HP_MOS8
