File: PCB/PDMS/pdms/voltage_out_mux.kicad_sch (KiCad schematic)
At the start: 19 parts, among them IC13 NX3L4051PW,118

Commit message: Update commit
Connections:
- net HP_MOS1: now also R154.2; no longer R136.2
- net HP_MOS3: now also R136.2; no longer R154.2
- net HP_MOS_DIV3: now reaches IC13.13 (Y0), R136.1, R138.2
- net HP_MOS_DIV7: now reaches IC13.2 (Y6), R139.1, R140.2
- net HP_MOS_DIV6: now reaches IC13.5 (Y5), R143.1, R152.2
- net HP_MOS_DIV8: now reaches IC13.4 (Y7), R134.1, R137.2
- net HP_MOS_DIV5: now reaches IC13.1 (Y4), R155.1, R156.2
- net HP_MOS_DIV1: now reaches IC13.15 (Y2), R153.2, R154.1
- net HP_MOS_DIV2: now reaches IC13.14 (Y1), R141.2, R142.1
- net HP_MOS_DIV4: now reaches IC13.12 (Y3), R157.2, R158.1
Changed lines of the file:
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@@
     (stroke (width 0) (type default) (color 0 0 0 0))
   )
-  (global_label "HP_MOS3" (shape input) (at 134.366 36.576 90) (fields_autoplaced)
+  (label "HP_MOS_DIV8" (at 109.855 73.66 0)
+    (effects (font (size 0.7 0.7)) (justify left bottom))
+  )
+  (label "HP_MOS_DIV4" (at 109.855 58.42 0)
+    (effects (font (size 0.7 0.7)) (justify left bottom))
+  )
+  (label "HP_MOS_DIV7" (at 109.855 69.85 0)
+    (effects (font (size 0.7 0.7)) (justify left bottom))
+  )
+  (label "HP_MOS_DIV1" (at 109.855 54.61 0)
+    (effects (font (size 0.7 0.7)) (justify left bottom))
+  )
+  (label "HP_MOS_DIV3" (at 109.855 46.99 0)
+    (effects (font (size 0.7 0.7)) (justify left bottom))
+  )
+  (label "HP_MOS_DIV2" (at 109.855 50.8 0)
+    (effects (font (size 0.7 0.7)) (justify left bottom))
+  )
+  (label "HP_MOS_DIV5" (at 109.855 62.23 0)
+    (effects (font (size 0.7 0.7)) (justify left bottom))
+  )
+  (label "HP_MOS_DIV6" (at 109.855 66.04 0)
+    (effects (font (size 0.7 0.7)) (justify left bottom))
+  )
+  (global_label "HP_MOS3" (shape input) (at 120.65 36.83 90) (fields_autoplaced)
     (effects (font (size 1.27 1.27)) (justify left))
-    (property "Intersheet References" "${INTERSHEET_REFS}" (id 0) (at 134.2866 25.3939 90)
+    (property "Intersheet References" "${INTERSHEET_REFS}" (id 0) (at 120.5706 25.6479 90)
       (effects (font (size 1.27 1.27)) (justify left) hide)
     )
@@
     )
   )
-  (global_label "HP_MOS1" (shape input) (at 120.65 36.83 90) (fields_autoplaced)
+  (global_label "HP_MOS1" (shape input) (at 134.366 36.576 90) (fields_autoplaced)
     (effects (font (size 1.27 1.27)) (justify left))
-    (property "Intersheet References" "${INTERSHEET_REFS}" (id 0) (at 120.5706 25.6479 90)
+    (property "Intersheet References" "${INTERSHEET_REFS}" (id 0) (at 134.2866 25.3939 90)
       (effects (font (size 1.27 1.27)) (justify left) hide)
     )

Commit message: Voltage mux finished
Connections:
- net HP_MOS_DIV5: now also IC13.5 (Y5); no longer IC13.1 (Y4)
- net HP_MOS_DIV6: now also IC13.4 (Y7); no longer IC13.5 (Y5)
- net HP_MOS_DIV8: now also IC13.1 (Y4); no longer IC13.4 (Y7)
Other:
- moved on the sheet: R134, R137, R143, R152, R155, R156

Commit message: Flash layout
Parts:
- C89: footprint Capacitor_SMD:C_0402_1005Metric_Pad0.74x0.62mm_HandSolder -> Capacitor_SMD:C_0402_1005Metric
Changed lines of the file:
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@@
     (property "Reference" "C89" (id 0) (at 104.14 32.385 90))
     (property "Value" "100nF" (id 1) (at 105.41 38.735 90))
-    (property "Footprint" "Capacitor_SMD:C_0402_1005Metric_Pad0.74x0.62mm_HandSolder" (id 2) (at 104.14 35.56 0)
+    (property "Footprint" "Capacitor_SMD:C_0402_1005Metric" (id 2) (at 104.14 35.56 0)
       (effects (font (size 1.27 1.27)) hide)
     )
