File: PCB/PDMS/pdms/hp_vmux.kicad_sch (KiCad schematic)
At the start: 20 parts, among them IC13 NX3L4051PW,118

Commit message: Finished layout - w/o stiching
Parts:
- removed C89: 100nF, Capacitor_SMD:C_0402_1005Metric, symbol Device:C_Small
- removed D38: BAT54SW, Package_TO_SOT_SMD:SOT-323_SC-70, symbol Diode:BAT54SW
- removed IC13: NX3L4051PW,118, PDMS_Additional:SOP65P640X110-16N, symbol pdms_additional:NX3L4051PW,118
- removed R134, R136, R139, R142, R143, R154, R155, R158: 10k, Resistor_SMD:R_0402_1005Metric, symbol Device:R_Small
- removed R135: 10, Resistor_SMD:R_0402_1005Metric, symbol Device:R_Small
- removed R137, R138, R140, R141, R152, R153, R156, R157: 2.3k, Resistor_SMD:R_0402_1005Metric, symbol Device:R_Small
