File: PCB/PDMS/pdms/lp_vmux.kicad_sch (KiCad schematic)
At the start: 20 parts, among them IC2 NX3L4051PW,118

Commit message: Finished layout - w/o stiching
Parts:
- removed C2: 100nF, Capacitor_SMD:C_0402_1005Metric, symbol Device:C_Small
- removed D42: BAT54SW, Package_TO_SOT_SMD:SOT-323_SC-70, symbol Diode:BAT54SW
- removed IC2: NX3L4051PW,118, PDMS_Additional:SOP65P640X110-16N, symbol pdms_additional:NX3L4051PW,118
- removed R10: 10, Resistor_SMD:R_0402_1005Metric, symbol Device:R_Small
- removed R11, R14, R15, R18, R19, R34, R35, R38: 10k, Resistor_SMD:R_0402_1005Metric, symbol Device:R_Small
- removed R12, R13, R16, R17, R32, R33, R36, R37: 2.3k, Resistor_SMD:R_0402_1005Metric, symbol Device:R_Small
